Commit message: Tidy files and change design

File: go2_like.urdf (robot description, URDF)
Before this commit: robot go2_like, 13 links, 12 joints
Links:
- link base_link: geometry collision box size=0.4 0.25 0.12; visual box size=0.08 0.18 0.08
- link fl_hip_link: geometry collision sphere radius=0.04; visual sphere radius=0.04
- link fl_shank_link: geometry collision cylinder length=0.04 radius=0.032; collision cylinder length=0.2 radius=0.022
- link fl_thigh_link: geometry collision cylinder length=0.2 radius=0.028; visual cylinder length=0.2 radius=0.028
- link fr_hip_link: geometry collision sphere radius=0.04; visual sphere radius=0.04
- link fr_shank_link: geometry collision cylinder length=0.04 radius=0.032; collision cylinder length=0.2 radius=0.022
- link fr_thigh_link: geometry collision cylinder length=0.2 radius=0.028; visual cylinder length=0.2 radius=0.028
- link rl_hip_link: geometry collision sphere radius=0.04; visual sphere radius=0.04
- link rl_shank_link: geometry collision cylinder length=0.04 radius=0.032; collision cylinder length=0.2 radius=0.022
- link rl_thigh_link: geometry collision cylinder length=0.2 radius=0.028; visual cylinder length=0.2 radius=0.028
- link rr_hip_link: geometry collision sphere radius=0.04; visual sphere radius=0.04
- link rr_shank_link: geometry collision cylinder length=0.04 radius=0.032; collision cylinder length=0.2 radius=0.022
- link rr_thigh_link: geometry collision cylinder length=0.2 radius=0.028; visual cylinder length=0.2 radius=0.028
